File: Hardware/V1.0.0/UF_MOT/iROB-EA_VS_2021_UF_MOT.sch (KiCad schematic (older format))
At the start: 2 parts

Commit message: Actualizacion general
Parts:
- removed U?: POLOLU-DRIVER-36v9, symbol POLOLU-DRIVER-36v9
- added C? (x2): 100uF/25V, symbol CP
- added C? (x2): 10uF/25V, symbol CP
- added M?: Motor_Derecho, symbol Motor_DC
- added M?: Motor_Izquierdo, symbol Motor_DC
- added R? (x3): 47K, symbol R
- added U?: 4051, symbol 4051
- added U?: POLOLU-DRIVER-36v9, symbol POLOLU-DRIVER-36v9
- added U? (x2): POLOLU_ACS714, symbol POLOLU_ACS714
- added U? (x2): LM7806ACT, TO-220, symbol LM7806ACT
Connections:
- net labels added: +12P, +5VA, GND, MTDI_INFO, MTDI_SEL_A, MTDI_SEL_B, MTDI_SEL_C, MTD_DIR, MTD_PWM, MTD_RESET, MTI_DIR, MTI_PWM, MTI_RESET
- wire segments 1 -> 96

Commit message: Actualizacion 2021
Parts:
- removed R? (x3): 47K, symbol R
- removed U? (x2): POLOLU_ACS714, symbol POLOLU_ACS714
Connections:
- net GND: now also U?.12 (X3), U?.13 (X0)
- net at C?.1, U?.~ (RESET): now also U?.3 (OUT) (x2)
Other:
- note added: "16"
- note added: "8"
- note added: "VCC"
- note added: "VSS"
Changed lines of the file:
@@
 	4400 2650 4450 2650
-Wire Wire Line
-	4450 1000 4450 5850
 Wire Wire Line
 	2900 2050 2850 2050
@@
 	8300 4350 8400 4350
 Wire Wire Line
-	8400 4350 8400 4800
+	8400 4150 8400 4800
 Wire Wire Line
 	8300 3250 8500 3250
@@
 Wire Wire Line
 	5000 3350 6900 3350
-$Comp
-L R R?
-U 1 1 60606131
-P 6600 4650
-F 0 "R?" V 6680 4650 50  0001 C CNN
-F 1 "47K" V 6600 4650 50  0000 C CNN
-F 2 "" V 6530 4650 50  0000 C CNN
-F 3 "" H 6600 4650 50  0000 C CNN
-	1    6600 4650
-	1    0    0    -1
-$EndComp
-$Comp
-L R R?
-U 1 1 606061A2
-P 6450 4650
-F 0 "R?" V 6530 4650 50  0001 C CNN
-F 1 "47K" V 6450 4650 50  0000 C CNN
-F 2 "" V 6380 4650 50  0000 C CNN
-F 3 "" H 6450 4650 50  0000 C CNN
-	1    6450 4650
-	1    0    0    -1
-$EndComp
-$Comp
-L R R?
-U 1 1 606061B0
-P 6300 4650
-F 0 "R?" V 6380 4650 50  0001 C CNN
-F 1 "47K" V 6300 4650 50  0000 C CNN
-F 2 "" V 6230 4650 50  0000 C CNN
-F 3 "" H 6300 4650 50  0000 C CNN
-	1    6300 4650
-	1    0    0    -1
-$EndComp
 Wire Wire Line
 	6900 4450 6600 4450
 Wire Wire Line
-	6600 2900 6600 4500
-Wire Wire Line
 	6900 4350 6450 4350
 Wire Wire Line
-	6450 2750 6450 4500
-Wire Wire Line
 	6900 4250 6300 4250
-Wire Wire Line
-	6300 2600 6300 4500
-$Comp
-L GND #PWR?
-U 1 1 6060622E
-P 6600 4850
-F 0 "#PWR?" H 6600 4600 50  0001 C CNN
-F 1 "GND" H 6600 4700 50  0001 C CNN
-F 2 "" H 6600 4850 50  0000 C CNN
-F 3 "" H 6600 4850 50  0000 C CNN
-	1    6600 4850
-	1    0    0    -1
-$EndComp
-$Comp
-L GND #PWR?
-U 1 1 6060623C
-P 6450 4850
-F 0 "#PWR?" H 6450 4600 50  0001 C CNN
-F 1 "GND" H 6450 4700 50  0001 C CNN
-F 2 "" H 6450 4850 50  0000 C CNN
-F 3 "" H 6450 4850 50  0000 C CNN
-	1    6450 4850
-	1    0    0    -1
-$EndComp
-$Comp
-L GND #PWR?
-U 1 1 6060624A
-P 6300 4850
-F 0 "#PWR?" H 6300 4600 50  0001 C CNN
-F 1 "GND" H 6300 4700 50  0001 C CNN
-F 2 "" H 6300 4850 50  0000 C CNN
-F 3 "" H 6300 4850 50  0000 C CNN
-	1    6300 4850
-	1    0    0    -1
-$EndComp
-Wire Wire Line
-	6600 4800 6600 4850
-Wire Wire Line
-	6450 4800 6450 4850
-Wire Wire Line
-	6300 4800 6300 4850
 $Comp
 L GND #PWR?
@@
 Wire Wire Line
 	8500 2900 6600 2900
-Connection ~ 6600 4450
 Wire Wire Line
 	6450 2750 8500 2750
-Connection ~ 6450 4350
 Wire Wire Line
 	8500 2600 6300 2600
-Connection ~ 6300 4250
 $Comp
 L POLOLU-DRIVER-36v9 U?
@@
 	2900 1950 2600 1950
 Wire Wire Line
-	2600 1150 2600 2750
+	2600 1000 2600 2750
 $Comp
 L GND #PWR?
@@
 Wire Wire Line
 	2600 3050 2600 3100
-$Comp
-L POLOLU_ACS714 U?
-U 1 1 60606ACB
-P 3300 800
-F 0 "U?" H 3150 750 39  0001 C CNN
-F 1 "POLOLU_ACS714" H 3350 800 39  0000 C CNN
-F 2 "" H 3300 800 39  0001 C CNN
-F 3 "" H 3300 800 39  0001 C CNN
-	1    3300 800
-	1    0    0    -1
-$EndComp
-Wire Wire Line
-	6900 3250 5200 3250
-Wire Wire Line
-	5200 3250 5200 1300
-Wire Wire Line
-	5200 1300 3800 1300
-Connection ~ 4450 2650
-Wire Wire Line
-	2900 1150 2600 1150
+Wire Wire Line
+	4700 3250 6900 3250
 Connection ~ 2600 1950
 Wire Wire Line
-	3800 1000 4450 1000
-$Comp
-L +5VA #PWR?
-U 1 1 60606D0D
-P 4700 1150
-F 0 "#PWR?" H 4700 1000 50  0001 C CNN
-F 1 "+5VA" V 4650 1400 50  0000 C CNN
-F 2 "" H 4700 1150 50  0000 C CNN
-F 3 "" H 4700 1150 50  0000 C CNN
-	1    4700 1150
-	0    1    1    0
-$EndComp
-Wire Wire Line
-	3800 1150 4700 1150
-$Comp
-L POLOLU_ACS714 U?
-U 1 1 60606D84
-P 3300 3450
-F 0 "U?" H 3150 3400 39  0001 C CNN
-F 1 "POLOLU_ACS714" H 3350 3450 39  0000 C CNN
-F 2 "" H 3300 3450 39  0001 C CNN
-F 3 "" H 3300 3450 39  0001 C CNN
-	1    3300 3450
-	1    0    0    -1
-$EndComp
-Connection ~ 4450 5250
-Wire Wire Line
-	6200 3950 6200 3550
-Wire Wire Line
-	6200 3550 6900 3550
+	4700 3550 6900 3550
 Wire Wire Line
 	5000 3650 5000 4750
@@
 	5100 4850 5100 3750
 Wire Wire Line
-	3800 3650 4450 3650
-Connection ~ 4450 3650
-Wire Wire Line
-	6200 3950 3800 3950
-Wire Wire Line
 	5000 4750 4400 4750
 Wire Wire Line
 	4400 4850 5100 4850
-Wire Wire Line
-	4550 1150 4550 3800
-Wire Wire Line
-	4550 3800 3800 3800
-Connection ~ 4550 1150
 $Comp
 L CP C?
@@
 	2600 5800 2600 5850
 Wire Wire Line
-	2900 3800 2600 3800
-Wire Wire Line
-	2600 3800 2600 5500
+	2600 3650 2600 5500
 Wire Wire Line
 	2900 4550 2600 4550
@@
 	1    0    0    -1
 $EndComp
-Wire Wire Line
-	2200 1000 2900 1000
 $Comp
 L GND #PWR?
@@
 	1400 3650 1400 3950
 Wire Wire Line
-	2250 3650 2900 3650
-Wire Wire Line
 	900  800  900  3650
 Connection ~ 1400 3650
@@
 $EndComp
 Connection ~ 900  1000
+Wire Wire Line
+	2200 1000 2600 1000
+Wire Wire Line
+	2250 3650 2600 3650
+$Comp
+L GND #PWR?
+U 1 1 6089B96B
+P 4700 3800
+F 0 "#PWR?" H 4700 3550 50  0001 C CNN
+F 1 "GND" H 4700 3650 50  0001 C CNN
+F 2 "" H 4700 3800 50  0000 C CNN
+F 3 "" H 4700 3800 50  0000 C CNN
+	1    4700 3800
+	1    0    0    -1
+$EndComp
+Wire Wire Line
+	4700 3250 4700 3800
+Connection ~ 4700 3550
+$Comp
+L GND #PWR?
+U 1 1 6089BA3C
+P 4450 3100
+F 0 "#PWR?" H 4450 2850 50  0001 C CNN
+F 1 "GND" H 4450 2950 50  0001 C CNN
+F 2 "" H 4450 3100 50  0000 C CNN
+F 3 "" H 4450 3100 50  0000 C CNN
+	1    4450 3100
+	1    0    0    -1
+$EndComp
+Wire Wire Line
+	4450 2650 4450 3100
+Wire Wire Line
+	4450 5250 4450 5850
+Wire Wire Line
+	6450 4350 6450 2750
+Wire Wire Line
+	6600 2900 6600 4450
+Wire Wire Line
+	6300 2600 6300 4250
+Text Notes 7800 4200 0    47   ~ 0
+VSS
+Wire Wire Line
+	8000 4150 8400 4150
+Connection ~ 8400 4350
+Text Notes 8150 4150 0    47   ~ 0
+8
+Text Notes 7800 4000 0    47   ~ 0
+VCC
+$Comp
+L +5VA #PWR?
+U 1 1 6089BD18
+P 8400 3950
+F 0 "#PWR?" H 8400 3800 50  0001 C CNN
+F 1 "+5VA" H 8400 4090 50  0000 C CNN
+F 2 "" H 8400 3950 50  0000 C CNN
+F 3 "" H 8400 3950 50  0000 C CNN
+	1    8400 3950
+	1    0    0    -1
+$EndComp
+Wire Wire Line
+	8000 3950 8400 3950
+Text Notes 8150 3950 0    47   ~ 0
+16
 $EndSCHEMATC
