File: Hardware/V1.0.0/UF_ENE/iROB-EA_VS_2021_UF_ENE.sch (KiCad schematic (older format))
At the start: 46 parts

Commit message: Actualizacion general
Parts:
- added C?: 10uF/16V, symbol CP
- added D?: 1N4007, symbol D
- added D? (x4): 24V, symbol D_Zener
- added R? (x2): 10ohm, symbol R
- added R?: 47K, symbol R
- added R?: 33K, symbol R
- added RL?: RE5V, symbol AZ850-x
Connections:
- net GND: now also C?.2, D?.1 (K), D?.1 (K), D?.2 (A), R?.1, RL?.10
- net at U?.3 (OUT12_VCC): now also RL?.9; no longer F?.2
- net at RL?.10, RL?.8: now also RL?.3; no longer RL?.3, U?.5 (OUT5V_VCC)
- new net: RL?.2, U?.5 (OUT5V_VCC)
- new net: F?.2, RL?.8
- new net: D?.2 (A), D?.2 (A) (x2)
- new net DBG-12V: RL?.7
- new net DBG-5V: D?.1 (K), R?.2, RL?.1, RL?.4
- new net DBG-RS232-RX-A: R?.2
- new net DBG-RS232-RX-B: D?.1 (K), R?.1
- new net DBG-RS232-TX-A: R?.2
- new net DBG-RS232-TX-B: D?.1 (K), R?.1
- new net DEBUG-ACTIVO: C?.1, R?.1, R?.2
Other:
- note added: "ALIMENTACION EXTERIOR (DEBUG)"
- note added: "ALIMENTACION MOTORES"
- note added: "ALIMENTACION PC"
- note added: "CONECTOR EXTERIOR\nDEBUG"
- moved on the sheet: F?

Commit message: Actualizacion python
Changed lines of the file:
@@
 Wire Notes Line
 	550  6700 550  5150
-Text GLabel 1450 5400 0    60   UnSpc ~ 0
-DBG-NC1
-Text GLabel 1450 5250 0    60   UnSpc ~ 0
-DBG-NC2
+Text GLabel 1450 5400 0    60   Output ~ 0
+DBG-RX
+Text GLabel 1450 5250 0    60   Input ~ 0
+DBG-TX
 Wire Notes Line
 	550  5150 1600 5150
